File: schematic_files/ZetaBot.kicad_pcb (KiCad board)
At the start: 2 copper layers, 241.5 x 110.5 mm, 23 parts, among them J1 USB C PD Modulle, J2 Conn_01x05, J3 MOTOR_L, J4 MOTOR_R, SW1 SW_SPDT, U1 RPI5, U1 RPLIDAR C1, U2 Buck Converter

Commit message: Added readme
Parts:
- removed the ? at (38.2, 121.2)
- removed the ? at (134.2, 121.6)
- removed the ? at (133.8, 61.2)
- removed the ? at (38.2, 61.2)
Other:
- board text added: "ζ"
- board text removed: "Δ"
Changed lines of the file:
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@@
 		(embedded_fonts no)
 	)
-	(footprint ""
-		(layer "F.Cu")
-		(at 38.2 121.2)
-		(property "Reference" ""
-			(at 0 0 0)
-			(layer "F.SilkS")
-			(effects
-				(font
-					(size 1.27 1.27)
-				)
-			)
-		)
-		(property "Value" ""
-			(at 0 0 0)
-			(layer "F.Fab")
-			(effects
-				(font
-					(size 1.27 1.27)
-				)
-			)
-		)
-		(property "Datasheet" ""
-			(at 0 0 0)
-			(layer "F.Fab")
-			(hide yes)
-			(effects
-				(font
-					(size 1.27 1.27)
-				)
-			)
-		)
-		(property "Description" ""
-			(at 0 0 0)
-			(layer "F.Fab")
-			(hide yes)
-			(effects
-				(font
-					(size 1.27 1.27)
-				)
-			)
-		)
-		(duplicate_pad_numbers_are_jumpers no)
-		(pad "" np_thru_hole circle
-			(at 4.8 -0.2 90)
-			(size 4 4)
-			(drill 4)
-			(layers "*.Cu" "*.Mask")
-			(thermal_bridge_angle 90)
-		)
-		(embedded_fonts no)
-	)
-	(footprint ""
-		(layer "F.Cu")
-		(at 134.2 121.6)
-		(property "Reference" ""
-			(at 0 0 0)
-			(layer "F.SilkS")
-			(effects
-				(font
-					(size 1.27 1.27)
-				)
-			)
-		)
-		(property "Value" ""
-			(at 0 0 0)
-			(layer "F.Fab")
-			(effects
-				(font
-					(size 1.27 1.27)
-				)
-			)
-		)
-		(property "Datasheet" ""
-			(at 0 0 0)
-			(layer "F.Fab")
-			(hide yes)
-			(effects
-				(font
-					(size 1.27 1.27)
-				)
-			)
-		)
-		(property "Description" ""
-			(at 0 0 0)
-			(layer "F.Fab")
-			(hide yes)
-			(effects
-				(font
-					(size 1.27 1.27)
-				)
-			)
-		)
-		(duplicate_pad_numbers_are_jumpers no)
-		(pad "" np_thru_hole circle
-			(at -1.2 -0.6 90)
-			(size 4 4)
-			(drill 4)
-			(layers "*.Cu" "*.Mask")
-			(thermal_bridge_angle 90)
-		)
-		(embedded_fonts no)
-	)
 	(footprint "ZetaBotFootprints:BUCK_CONV"
 		(layer "F.Cu")
@@
 		(embedded_fonts no)
 	)
-	(footprint ""
-		(layer "F.Cu")
-		(at 133.8 61.2)
-		(property "Reference" ""
-			(at 0 0 0)
-			(layer "F.SilkS")
-			(effects
-				(font
-					(size 1.27 1.27)
-				)
-			)
-		)
-		(property "Value" ""
-			(at 0 0 0)
-			(layer "F.Fab")
-			(effects
-				(font
-					(size 1.27 1.27)
-				)
-			)
-		)
-		(property "Datasheet" ""
-			(at 0 0 0)
-			(layer "F.Fab")
-			(hide yes)
-			(effects
-				(font
-					(size 1.27 1.27)
-				)
-			)
-		)
-		(property "Description" ""
-			(at 0 0 0)
-			(layer "F.Fab")
-			(hide yes)
-			(effects
-				(font
-					(size 1.27 1.27)
-				)
-			)
-		)
-		(duplicate_pad_numbers_are_jumpers no)
-		(pad "" np_thru_hole circle
-			(at -0.8 -0.2 90)
-			(size 4 4)
-			(drill 4)
-			(layers "*.Cu" "*.Mask")
-			(thermal_bridge_angle 90)
-		)
-		(embedded_fonts no)
-	)
 	(footprint "deltabot:C_Disc_D3.0mm_W2.0mm_P2.50mm"
 		(layer "F.Cu")
@@
 		)
 	)
-	(footprint ""
-		(layer "F.Cu")
-		(at 38.2 61.2)
-		(property "Reference" ""
-			(at 0 0 0)
-			(layer "F.SilkS")
-			(effects
-				(font
-					(size 1.27 1.27)
-				)
-			)
-		)
-		(property "Value" ""
-			(at 0 0 0)
-			(layer "F.Fab")
-			(effects
-				(font
-					(size 1.27 1.27)
-				)
-			)
-		)
-		(property "Datasheet" ""
-			(at 0 0 0)
-			(layer "F.Fab")
-			(hide yes)
-			(effects
-				(font
-					(size 1.27 1.27)
-				)
-			)
-		)
-		(property "Description" ""
-			(at 0 0 0)
-			(layer "F.Fab")
-			(hide yes)
-			(effects
-				(font
-					(size 1.27 1.27)
-				)
-			)
-		)
-		(duplicate_pad_numbers_are_jumpers no)
-		(pad "" np_thru_hole circle
-			(at 4.8 -0.2 90)
-			(size 4 4)
-			(drill 4)
-			(layers "*.Cu" "*.Mask")
-			(thermal_bridge_angle 90)
-		)
-		(embedded_fonts no)
-	)
 	(footprint "deltabot:C_Disc_D3.0mm_W2.0mm_P2.50mm"
 		(layer "F.Cu")
@@
 		)
 	)
-	(gr_text "Δ\n"
-		(at 266 44 90)
+	(gr_text "ζ"
+		(at 264.5 44 90)
 		(layer "F.Cu")
 		(effects
 			(font
-				(size 5 4)
+				(size 4 4)
 				(thickness 0.8)
 				(bold yes)
@@
 	)
 	(segment
-		(start 191.5 66.5)
-		(end 191.5 68)
-		(width 1)
-		(layer "F.Cu")
-		(net "PWM_L")
-	)
-	(segment
-		(start 184 75.5)
-		(end 76.9 75.5)
-		(width 1)
-		(layer "F.Cu")
-		(net "PWM_L")
-	)
-	(segment
-		(start 191.5 68)
-		(end 184 75.5)
-		(width 1)
-		(layer "F.Cu")
-		(net "PWM_L")
-	)
-	(segment
-		(start 75.005 73.605)
-		(end 72.5125 73.605)
-		(width 1)
-		(layer "F.Cu")
-		(net "PWM_L")
-	)
-	(segment
-		(start 76.9 75.5)
-		(end 75.005 73.605)
-		(width 1)
-		(layer "F.Cu")
-		(net "PWM_L")
-	)
-	(segment
-		(start 191.5 66.5)
-		(end 201.5 66.5)
-		(width 1)
-		(layer "F.Cu")
-		(net "PWM_L")
-	)
-	(segment
 		(start 159 100)
 		(end 151 108)
@@
 	)
 	(segment
+		(start 194.699 138)
+		(end 194.699 132.199)
+		(width 2)
+		(layer "B.Cu")
+		(net "Net-(SW1-B)")
+	)
+	(segment
+		(start 191.2 128.7)
+		(end 189.6 128.7)
+		(width 2)
+		(layer "B.Cu")
+		(net "Net-(SW1-B)")
+	)
+	(segment
+		(start 194.699 132.199)
+		(end 191.2 128.7)
+		(width 2)
+		(layer "B.Cu")
+		(net "Net-(SW1-B)")
+	)
+	(segment
 		(start 50 75.8)
 		(end 52.2 73.6)
@@
 	)
 	(segment
-		(start 194.699 138)
-		(end 194.699 132.199)
-		(width 2)
-		(layer "B.Cu")
-		(net "Net-(SW1-B)")
+		(start 191.5 66.5)
+		(end 191.5 68)
+		(width 1)
+		(layer "F.Cu")
+		(net "PWM_L")
 	)
 	(segment
-		(start 191.2 128.7)
-		(end 189.6 128.7)
-		(width 2)
-		(layer "B.Cu")
-		(net "Net-(SW1-B)")
+		(start 184 75.5)
+		(end 76.9 75.5)
+		(width 1)
+		(layer "F.Cu")
+		(net "PWM_L")
 	)
 	(segment
-		(start 194.699 132.199)
-		(end 191.2 128.7)
-		(width 2)
-		(layer "B.Cu")
-		(net "Net-(SW1-B)")
+		(start 191.5 68)
+		(end 184 75.5)
+		(width 1)
+		(layer "F.Cu")
+		(net "PWM_L")
+	)
+	(segment
+		(start 75.005 73.605)
+		(end 72.5125 73.605)
+		(width 1)
+		(layer "F.Cu")
+		(net "PWM_L")
+	)
+	(segment
+		(start 76.9 75.5)
+		(end 75.005 73.605)
+		(width 1)
+		(layer "F.Cu")
+		(net "PWM_L")
+	)
+	(segment
+		(start 191.5 66.5)
+		(end 201.5 66.5)
+		(width 1)
+		(layer "F.Cu")
+		(net "PWM_L")
 	)
 	(zone
